File: pcb.kicad_sch (KiCad schematic)
At the start: 3 parts

Commit message: hopefully fix example :/
Parts:
- BT1: footprint Battery:BatteryHolder_Keystone_1057_1x2032 -> Battery:BatteryHolder_Keystone_3034_1x20mm
Changed lines of the file:
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@@
       (effects (font (size 1.27 1.27)) (justify left))
     )
-    (property "Footprint" "Battery:BatteryHolder_Keystone_1057_1x2032" (at 133.35 100.076 90)
+    (property "Footprint" "Battery:BatteryHolder_Keystone_3034_1x20mm" (at 133.35 100.076 90)
       (effects (font (size 1.27 1.27)) hide)
     )
